File: Reflow-A-Tron/Reflow-A-Tron.brd (EAGLE design)
At the start: 97.8 x 62.2 mm, 40 parts, among them IC1 ATMEGA644-10PU, J2 HOT, J3 NEUTRAL, Q1 FOXSLF/200-20, Q2 BSS123, U2 MC7805, U4 MAX6675

Commit message: Name
Parts:
- U2: value MC7805 -> L4941BDT-TRDPAK-3
Other:
- board text added: "C:/Users/Neil/eagle-stuff/Reflow-A-Tron/ReflowTron.bmp"
- board text added: "v1.0"
