File: Reflow-A-Tron/Reflow-A-Tron.sch (EAGLE design)
At the start: 40 parts, among them IC1 ATMEGA644-10PU, J2 HOT, J3 NEUTRAL, Q1 FOXSLF/200-20, Q2 BSS123, U1 FT230X, U2 L4941BDT-TRDPAK-3, U4 MAX6675

Commit message: Fix shit
Parts:
- added R12: 10k, resistor:R-US_R0805
Connections:
- removed net GND-MCU: C6.2, C7.1, C8.1, IC1.GND, IC1.GND@1
- removed net VCC-MCU: C6.1, IC1.AREF, IC1.AVCC, IC1.VCC
- net 5V: now also C6.1, IC1.AREF, IC1.AVCC, IC1.VCC
- net GND: now also C6.2, C7.1, C8.1, IC1.GND, IC1.GND@1, R12.2
- net TRIAC-CTRL: now also R12.1
Other:
- moved on the sheet: C6
Changed lines of the file:
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@@
 <part name="GND4" library="SparkFun-Aesthetics" deviceset="GND" device=""/>
 <part name="C6" library="SparkFun-Capacitors" deviceset="0.1UF-25V(+80/-20%)(0603)" device="" value="0.1uF"/>
-<part name="GND5" library="SparkFun-Aesthetics" deviceset="GND" device=""/>
 <part name="SUPPLY6" library="SparkFun-Aesthetics" deviceset="5V" device=""/>
 <part name="Q1" library="crystal" deviceset="CRYSTAL" device="HC49S" value="FOXSLF/200-20"/>
@@
 <part name="D3" library="neilbetham" deviceset="T1250H" device=""/>
 <part name="OK1" library="optocoupler" deviceset="IL420" device=""/>
-<part name="GND9" library="SparkFun-Aesthetics" deviceset="GND" device=""/>
 <part name="R8" library="resistor" deviceset="R-US_" device="R0805" value="180"/>
 <part name="R9" library="resistor" deviceset="R-US_" device="R0805" value="2.2k"/>
@@
 <part name="J2" library="neilbetham" deviceset="8191" device="" value="HOT"/>
 <part name="J3" library="neilbetham" deviceset="8191" device="" value="NEUTRAL"/>
+<part name="GND10" library="SparkFun-Aesthetics" deviceset="GND" device=""/>
+<part name="R12" library="resistor" deviceset="R-US_" device="R0805" value="10k"/>
+<part name="GND5" library="SparkFun-Aesthetics" deviceset="GND" device=""/>
 </parts>
 <sheets>
@@
 <instance part="S1" gate="S" x="-53.34" y="60.96"/>
 <instance part="GND4" gate="1" x="-58.42" y="53.34"/>
-<instance part="C6" gate="G$1" x="-58.42" y="33.02"/>
-<instance part="GND5" gate="1" x="-60.96" y="25.4"/>
+<instance part="C6" gate="G$1" x="-55.88" y="33.02"/>
 <instance part="SUPPLY6" gate="G$1" x="-60.96" y="40.64"/>
 <instance part="Q1" gate="G$1" x="-58.42" y="10.16"/>
@@
 <instance part="D3" gate="G$1" x="307.34" y="35.56" rot="MR0"/>
 <instance part="OK1" gate="G$1" x="220.98" y="35.56"/>
-<instance part="GND9" gate="1" x="198.12" y="7.62"/>
 <instance part="R8" gate="G$1" x="251.46" y="48.26"/>
 <instance part="R9" gate="G$1" x="279.4" y="48.26"/>
@@
 <instance part="J2" gate="G$1" x="322.58" y="48.26"/>
 <instance part="J3" gate="G$1" x="322.58" y="15.24"/>
+<instance part="GND10" gate="1" x="-60.96" y="25.4" rot="MR0"/>
+<instance part="R12" gate="G$1" x="190.5" y="7.62" rot="R270"/>
+<instance part="GND5" gate="1" x="195.58" y="-5.08"/>
 </instances>
 <busses>
@@
 <pinref part="SUPPLY6" gate="G$1" pin="5V"/>
 <wire x1="-60.96" y1="40.64" x2="-60.96" y2="38.1" width="0.1524" layer="91"/>
-<wire x1="-60.96" y1="38.1" x2="-58.42" y2="38.1" width="0.1524" layer="91"/>
+<pinref part="C6" gate="G$1" pin="1"/>
+<wire x1="-55.88" y1="38.1" x2="-48.26" y2="38.1" width="0.1524" layer="91"/>
+<label x="-48.26" y="38.1" size="1.778" layer="95"/>
+<wire x1="-60.96" y1="38.1" x2="-55.88" y2="38.1" width="0.1524" layer="91"/>
+</segment>
+<segment>
+<pinref part="IC1" gate="G$1" pin="VCC"/>
+<wire x1="0" y1="50.8" x2="-2.54" y2="50.8" width="0.1524" layer="91"/>
+<label x="-12.7" y="50.8" size="1.778" layer="95"/>
+</segment>
+<segment>
+<pinref part="IC1" gate="G$1" pin="AREF"/>
+<wire x1="60.96" y1="53.34" x2="63.5" y2="53.34" width="0.1524" layer="91"/>
+<label x="63.5" y="53.34" size="1.778" layer="95"/>
+</segment>
+<segment>
+<pinref part="IC1" gate="G$1" pin="AVCC"/>
+<wire x1="60.96" y1="48.26" x2="63.5" y2="48.26" width="0.1524" layer="91"/>
+<label x="63.5" y="48.26" size="1.778" layer="95"/>
 </segment>
 </net>
@@
 <wire x1="175.26" y1="-10.16" x2="175.26" y2="-15.24" width="0.1524" layer="91"/>
 <wire x1="157.48" y1="-10.16" x2="175.26" y2="-10.16" width="0.1524" layer="91"/>
+<junction x="175.26" y="-10.16"/>
+</segment>
+<segment>
+<pinref part="C6" gate="G$1" pin="2"/>
+<wire x1="-55.88" y1="30.48" x2="-48.26" y2="30.48" width="0.1524" layer="91"/>
+<wire x1="-55.88" y1="30.48" x2="-60.96" y2="30.48" width="0.1524" layer="91"/>
+<label x="-48.26" y="30.48" size="1.778" layer="95"/>
+<pinref part="GND10" gate="1" pin="GND"/>
+<wire x1="-60.96" y1="30.48" x2="-60.96" y2="27.94" width="0.1524" layer="91"/>
 </segment>
 <segment>
 <pinref part="Q2" gate="G$1" pin="S"/>
-<pinref part="GND9" gate="1" pin="GND"/>
-<wire x1="198.12" y1="12.7" x2="198.12" y2="10.16" width="0.1524" layer="91"/>
-</segment>
-</net>
-<net name="RESET" class="0">
-<segment>
-<pinref part="S1" gate="S" pin="4"/>
-<pinref part="S1" gate="S" pin="3"/>
-<wire x1="-48.26" y1="58.42" x2="-48.26" y2="60.96" width="0.1524" layer="91"/>
-<wire x1="-48.26" y1="60.96" x2="-45.72" y2="60.96" width="0.1524" layer="91"/>
-<label x="-45.72" y="60.96" size="1.778" layer="95"/>
-</segment>
-<segment>
-<pinref part="IC1" gate="G$1" pin="!RESET"/>
-<wire x1="0" y1="53.34" x2="-2.54" y2="53.34" width="0.1524" layer="91"/>
-<label x="-17.78" y="53.34" size="1.778" layer="95"/>
-</segment>
-<segment>
-<pinref part="JP2" gate="G$1" pin="6"/>
-<wire x1="157.48" y1="-5.08" x2="160.02" y2="-5.08" width="0.1524" layer="91"/>
-<label x="160.02" y="-5.08" size="1.778" layer="95"/>
-</segment>
-</net>
-<net name="VCC-MCU" class="0">
-<segment>
-<pinref part="C6" gate="G$1" pin="1"/>
-<wire x1="-58.42" y1="38.1" x2="-48.26" y2="38.1" width="0.1524" layer="91"/>
-<label x="-48.26" y="38.1" size="1.778" layer="95"/>
-</segment>
-<segment>
-<pinref part="IC1" gate="G$1" pin="VCC"/>
-<wire x1="0" y1="50.8" x2="-2.54" y2="50.8" width="0.1524" layer="91"/>
-<label x="-17.78" y="50.8" size="1.778" layer="95"/>
-</segment>
-<segment>
-<pinref part="IC1" gate="G$1" pin="AREF"/>
-<wire x1="60.96" y1="53.34" x2="63.5" y2="53.34" width="0.1524" layer="91"/>
-<label x="63.5" y="53.34" size="1.778" layer="95"/>
-</segment>
-<segment>
-<pinref part="IC1" gate="G$1" pin="AVCC"/>
-<wire x1="60.96" y1="48.26" x2="63.5" y2="48.26" width="0.1524" layer="91"/>
-<label x="63.5" y="48.26" size="1.778" layer="95"/>
-</segment>
-</net>
-<net name="GND-MCU" class="0">
+<wire x1="198.12" y1="12.7" x2="198.12" y2="0" width="0.1524" layer="91"/>
+<pinref part="R12" gate="G$1" pin="2"/>
+<wire x1="198.12" y1="0" x2="195.58" y2="0" width="0.1524" layer="91"/>
+<wire x1="195.58" y1="0" x2="190.5" y2="0" width="0.1524" layer="91"/>
+<wire x1="190.5" y1="0" x2="190.5" y2="2.54" width="0.1524" layer="91"/>
+<pinref part="GND5" gate="1" pin="GND"/>
+<wire x1="195.58" y1="-2.54" x2="195.58" y2="0" width="0.1524" layer="91"/>
+<junction x="195.58" y="0"/>
+</segment>
 <segment>
 <pinref part="IC1" gate="G$1" pin="GND"/>
 <wire x1="0" y1="48.26" x2="-2.54" y2="48.26" width="0.1524" layer="91"/>
-<label x="-17.78" y="48.26" size="1.778" layer="95"/>
-</segment>
-<segment>
-<pinref part="IC1" gate="G$1" pin="GND@1"/>
-<wire x1="60.96" y1="50.8" x2="63.5" y2="50.8" width="0.1524" layer="91"/>
-<label x="63.5" y="50.8" size="1.778" layer="95"/>
+<label x="-12.7" y="48.26" size="1.778" layer="95"/>
 </segment>
 <segment>
@@
 </segment>
 <segment>
-<pinref part="C6" gate="G$1" pin="2"/>
-<wire x1="-58.42" y1="30.48" x2="-48.26" y2="30.48" width="0.1524" layer="91"/>
-<label x="-48.26" y="30.48" size="1.778" layer="95"/>
-<pinref part="GND5" gate="1" pin="GND"/>
-<wire x1="-58.42" y1="30.48" x2="-60.96" y2="30.48" width="0.1524" layer="91"/>
-<wire x1="-60.96" y1="30.48" x2="-60.96" y2="27.94" width="0.1524" layer="91"/>
+<pinref part="IC1" gate="G$1" pin="GND@1"/>
+<wire x1="60.96" y1="50.8" x2="63.5" y2="50.8" width="0.1524" layer="91"/>
+<label x="63.5" y="50.8" size="1.778" layer="95"/>
+</segment>
+</net>
+<net name="RESET" class="0">
+<segment>
+<pinref part="S1" gate="S" pin="4"/>
+<pinref part="S1" gate="S" pin="3"/>
+<wire x1="-48.26" y1="58.42" x2="-48.26" y2="60.96" width="0.1524" layer="91"/>
+<wire x1="-48.26" y1="60.96" x2="-45.72" y2="60.96" width="0.1524" layer="91"/>
+<label x="-45.72" y="60.96" size="1.778" layer="95"/>
+</segment>
+<segment>
+<pinref part="IC1" gate="G$1" pin="!RESET"/>
+<wire x1="0" y1="53.34" x2="-2.54" y2="53.34" width="0.1524" layer="91"/>
+<label x="-12.7" y="53.34" size="1.778" layer="95"/>
+</segment>
+<segment>
+<pinref part="JP2" gate="G$1" pin="6"/>
+<wire x1="157.48" y1="-5.08" x2="160.02" y2="-5.08" width="0.1524" layer="91"/>
+<label x="160.02" y="-5.08" size="1.778" layer="95"/>
 </segment>
 </net>
@@
 <pinref part="IC1" gate="G$1" pin="XTAL2"/>
 <wire x1="0" y1="45.72" x2="-2.54" y2="45.72" width="0.1524" layer="91"/>
-<label x="-17.78" y="45.72" size="1.778" layer="95"/>
+<label x="-12.7" y="45.72" size="1.778" layer="95"/>
 </segment>
 </net>
@@
 <pinref part="IC1" gate="G$1" pin="XTAL1"/>
 <wire x1="0" y1="43.18" x2="-2.54" y2="43.18" width="0.1524" layer="91"/>
-<label x="-17.78" y="43.18" size="1.778" layer="95"/>
+<label x="-12.7" y="43.18" size="1.778" layer="95"/>
 </segment>
 </net>
@@
 <pinref part="Q2" gate="G$1" pin="G"/>
 <wire x1="193.04" y1="15.24" x2="190.5" y2="15.24" width="0.1524" layer="91"/>
-<label x="172.72" y="15.24" size="1.778" layer="95"/>
-</segment>
-</net>
+<label x="170.18" y="15.24" size="1.778" layer="95"/>
+<pinref part="R12" gate="G$1" pin="1"/>
+<wire x1="190.5" y1="15.24" x2="185.42" y2="15.24" width="0.1524" layer="91"/>
+<wire x1="190.5" y1="15.24" x2="190.5" y2="12.7" width="0.1524" layer="91"/>
+<junction x="190.5" y="15.24"/>
+</segment>
+</net>

Commit message: More fixes
Connections:
- net N$10 renamed RXD
- net N$9 renamed TXD
Changed lines of the file:
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@@
 <?xml version="1.0" encoding="utf-8"?>
 <!DOCTYPE eagle SYSTEM "eagle.dtd">
-<eagle version="7.2.0">
+<eagle version="7.7.0">
 <drawing>
 <settings>
@@
 </segment>
 </net>
-<net name="N$9" class="0">
+<net name="TXD" class="0">
 <segment>
 <pinref part="IC1" gate="G$1" pin="PCINT24/RXD0_PD0"/>
@@
 <wire x1="71.12" y1="5.08" x2="71.12" y2="-20.32" width="0.1524" layer="91"/>
 <wire x1="71.12" y1="-20.32" x2="58.42" y2="-20.32" width="0.1524" layer="91"/>
-</segment>
-</net>
-<net name="N$10" class="0">
+<label x="63.5" y="-20.32" size="1.778" layer="95"/>
+</segment>
+</net>
+<net name="RXD" class="0">
 <segment>
 <pinref part="IC1" gate="G$1" pin="PCINT25/TXD0_PD1"/>
@@
 <wire x1="58.42" y1="-22.86" x2="73.66" y2="-22.86" width="0.1524" layer="91"/>
 <wire x1="73.66" y1="-22.86" x2="73.66" y2="7.62" width="0.1524" layer="91"/>
-</segment>
-</net>
+<label x="63.5" y="-25.4" size="1.778" layer="95"/>
+</segment>
+</net>

Commit message: Add custom lib, still needs more work.
Parts:
- C5, C6: value 0.1uF -> 10nF; device SparkFun-Capacitors:0.1UF-25V(+80/-20%)(0603) -> custom:SMD-CAP-0805
- J1: device neilbetham:XM7D-0512 -> custom:XM7D-0512
- U1: device neilbetham:FT230X -> custom:FT230X
Connections:
- removed net ID: J1.ID
- removed net MAX-SCK: IC1.PCINT15/SCK_PB7
- removed net MOSI: IC1.PCINT13/MOSI_PB5
- removed net N$1: C5.1, U4.VCC
- removed net N$2: IC1.PCINT12/OC0B/SS_PB4
- net 5V: now also C5.1, U4.VCC
- net CS: now also IC1.PCINT12/OC0B/SS_PB4
- net SCK: now also IC1.PCINT15/SCK_PB7
Changed lines of the file:
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@@
 <layer number="49" name="Reference" color="7" fill="1" visible="no" active="no"/>
 <layer number="50" name="dxf" color="7" fill="1" visible="no" active="no"/>
-<layer number="51" name="tDocu" color="6" fill="9" visible="no" active="no"/>
+<layer number="51" name="tDocu" color="7" fill="1" visible="no" active="no"/>
 <layer number="52" name="bDocu" color="7" fill="1" visible="no" active="no"/>
 <layer number="53" name="tGND_GNDA" color="7" fill="9" visible="no" active="no"/>
@@
 <part name="C2" library="SparkFun-Capacitors" deviceset="10UF50V20%(1210)" device="" value="10uF"/>
 <part name="GND3" library="SparkFun-Aesthetics" deviceset="GND" device=""/>
-<part name="C5" library="SparkFun-Capacitors" deviceset="0.1UF-25V(+80/-20%)(0603)" device="" value="0.1uF"/>
+<part name="C5" library="custom" deviceset="SMD-CAP" device="-0805" value="10nF"/>
 <part name="S1" library="SparkFun-Retired" deviceset="TAC_SWITCH" device="PTH"/>
 <part name="GND4" library="SparkFun-Aesthetics" deviceset="GND" device=""/>
-<part name="C6" library="SparkFun-Capacitors" deviceset="0.1UF-25V(+80/-20%)(0603)" device="" value="0.1uF"/>
+<part name="C6" library="custom" deviceset="SMD-CAP" device="-0805" value="10nF"/>
 <part name="SUPPLY6" library="SparkFun-Aesthetics" deviceset="5V" device=""/>
 <part name="Q1" library="crystal" deviceset="CRYSTAL" device="HC49S" value="FOXSLF/200-20"/>
@@
 <part name="SUPPLY7" library="SparkFun-Aesthetics" deviceset="VCC" device=""/>
 <part name="GND7" library="SparkFun-Aesthetics" deviceset="GND" device=""/>
-<part name="U1" library="neilbetham" deviceset="FT230X" device="" value="FT230X"/>
-<part name="J1" library="neilbetham" deviceset="XM7D-0512" device=""/>
+<part name="U1" library="custom" deviceset="FT230X" device="" value="FT230X"/>
+<part name="J1" library="custom" deviceset="XM7D-0512" device=""/>
 <part name="GND8" library="SparkFun-Aesthetics" deviceset="GND" device=""/>
 <part name="C3" library="neilbetham" deviceset="SMD-CAP" device="-0805" value="100nF"/>
@@
 <text x="198.12" y="152.4" size="1.778" layer="97">DC Low Voltage</text>
 <text x="220.98" y="152.4" size="1.778" layer="97">AC High Voltage</text>
+<wire x1="218.44" y1="162.56" x2="218.44" y2="-63.5" width="0.1524" layer="97" style="shortdash"/>
 </plain>
 <instances>
@@
 </instances>
 <busses>
-<bus name="SPI">
+<bus name="CS,MISO,SCK">
 <segment>
 <wire x1="-17.78" y1="58.42" x2="-17.78" y2="93.98" width="0.762" layer="92"/>
@@
 </segment>
 </bus>
-<bus name="USB">
+<bus name="USB-VCC,DP,DM,GND">
 <segment>
 <wire x1="12.7" y1="-43.18" x2="12.7" y2="-22.86" width="0.762" layer="92"/>
@@
 <pinref part="C1" gate="G$1" pin="1"/>
 <wire x1="2.54" y1="132.08" x2="2.54" y2="127" width="0.1524" layer="91"/>
+<junction x="2.54" y="132.08"/>
 </segment>
 <segment>
@@
 <pinref part="C2" gate="G$1" pin="1"/>
 <wire x1="33.02" y1="127" x2="33.02" y2="132.08" width="0.1524" layer="91"/>
+<junction x="33.02" y="132.08"/>
 </segment>
 <segment>
@@
 <wire x1="198.12" y1="53.34" x2="203.2" y2="53.34" width="0.1524" layer="91"/>
 <wire x1="198.12" y1="55.88" x2="198.12" y2="53.34" width="0.1524" layer="91"/>
+<junction x="198.12" y="53.34"/>
 </segment>
 <segment>
@@
 <wire x1="-60.96" y1="40.64" x2="-60.96" y2="38.1" width="0.1524" layer="91"/>
 <pinref part="C6" gate="G$1" pin="1"/>
-<wire x1="-55.88" y1="38.1" x2="-48.26" y2="38.1" width="0.1524" layer="91"/>
+<wire x1="-55.88" y1="30.48" x2="-48.26" y2="38.1" width="0.1524" layer="91"/>
 <label x="-48.26" y="38.1" size="1.778" layer="95"/>
-<wire x1="-60.96" y1="38.1" x2="-55.88" y2="38.1" width="0.1524" layer="91"/>
+<wire x1="-60.96" y1="38.1" x2="-55.88" y2="30.48" width="0.1524" layer="91"/>
+<junction x="-55.88" y="30.48"/>
 </segment>
 <segment>
@@
 <wire x1="60.96" y1="48.26" x2="63.5" y2="48.26" width="0.1524" layer="91"/>
 <label x="63.5" y="48.26" size="1.778" layer="95"/>
+</segment>
+<segment>
+<wire x1="116.84" y1="78.74" x2="116.84" y2="66.04" width="0.1524" layer="91"/>
+<wire x1="116.84" y1="66.04" x2="124.46" y2="73.66" width="0.1524" layer="91"/>
+<pinref part="C5" gate="G$1" pin="1"/>
+<junction x="116.84" y="66.04"/>
+<pinref part="U4" gate="G$1" pin="VCC"/>
+<pinref part="SUPPLY1" gate="G$1" pin="5V"/>
 </segment>
 </net>
@@
 <wire x1="17.78" y1="116.84" x2="33.02" y2="116.84" width="0.1524" layer="91"/>
 <wire x1="33.02" y1="116.84" x2="33.02" y2="119.38" width="0.1524" layer="91"/>
+<junction x="17.78" y="116.84"/>
 </segment>
 <segment>
 <pinref part="GND3" gate="1" pin="GND"/>
-<wire x1="124.46" y1="66.04" x2="116.84" y2="66.04" width="0.1524" layer="91"/>
-<wire x1="116.84" y1="66.04" x2="106.68" y2="66.04" width="0.1524" layer="91"/>
+<wire x1="124.46" y1="66.04" x2="116.84" y2="71.12" width="0.1524" layer="91"/>
+<wire x1="116.84" y1="71.12" x2="106.68" y2="66.04" width="0.1524" layer="91"/>
 <wire x1="106.68" y1="66.04" x2="106.68" y2="63.5" width="0.1524" layer="91"/>
 <pinref part="C5" gate="G$1" pin="2"/>
-<junction x="116.84" y="66.04"/>
+<junction x="116.84" y="71.12"/>
 <pinref part="U4" gate="G$1" pin="GND"/>
 </segment>
@@
 <pinref part="GND4" gate="1" pin="GND"/>
 <wire x1="-58.42" y1="58.42" x2="-58.42" y2="55.88" width="0.1524" layer="91"/>
+<junction x="-58.42" y="58.42"/>
 </segment>
 <segment>
@@
 <wire x1="-45.72" y1="-40.64" x2="-43.18" y2="-38.1" width="0.1524" layer="91"/>
 <label x="-60.96" y="-43.18" size="1.778" layer="95"/>
+<junction x="-53.34" y="-40.64"/>
 </segment>
 <segment>
@@
 <segment>
 <pinref part="C6" gate="G$1" pin="2"/>
-<wire x1="-55.88" y1="30.48" x2="-48.26" y2="30.48" width="0.1524" layer="91"/>
-<wire x1="-55.88" y1="30.48" x2="-60.96" y2="30.48" width="0.1524" layer="91"/>
+<wire x1="-55.88" y1="35.56" x2="-48.26" y2="30.48" width="0.1524" layer="91"/>
+<wire x1="-55.88" y1="35.56" x2="-60.96" y2="30.48" width="0.1524" layer="91"/>
 <label x="-48.26" y="30.48" size="1.778" layer="95"/>
 <pinref part="GND10" gate="1" pin="GND"/>
 <wire x1="-60.96" y1="30.48" x2="-60.96" y2="27.94" width="0.1524" layer="91"/>
+<junction x="-55.88" y="35.56"/>
 </segment>
 <segment>
@@
 <wire x1="-48.26" y1="60.96" x2="-45.72" y2="60.96" width="0.1524" layer="91"/>
 <label x="-45.72" y="60.96" size="1.778" layer="95"/>
+<junction x="-48.26" y="60.96"/>
 </segment>
 <segment>
@@
 <pinref part="THERMOCOUPLE" gate="G$1" pin="1"/>
 <wire x1="121.92" y1="45.72" x2="132.08" y2="45.72" width="0.1524" layer="91"/>
+<junction x="121.92" y="45.72"/>
 </segment>
 </net>
@@
 <pinref part="THERMOCOUPLE" gate="G$1" pin="2"/>
 <wire x1="129.54" y1="43.18" x2="132.08" y2="43.18" width="0.1524" layer="91"/>
-</segment>
-</net>
-<net name="MAX-SCK" class="0">
-<segment>
+<junction x="121.92" y="40.64"/>
+</segment>
+</net>
+<net name="SCK" class="0">
+<segment>
+<wire x1="-17.78" y1="58.42" x2="-15.24" y2="55.88" width="0.1524" layer="91"/>
+<wire x1="-15.24" y1="55.88" x2="0" y2="55.88" width="0.1524" layer="91"/>
+<label x="-15.24" y="55.88" size="1.778" layer="95"/>
 <pinref part="IC1" gate="G$1" pin="PCINT15/SCK_PB7"/>
-<wire x1="0" y1="55.88" x2="-2.54" y2="55.88" width="0.1524" layer="91"/>
-</segment>
-</net>
-<net name="N$1" class="0">
-<segment>
-<wire x1="116.84" y1="78.74" x2="116.84" y2="73.66" width="0.1524" layer="91"/>
-<wire x1="116.84" y1="73.66" x2="124.46" y2="73.66" width="0.1524" layer="91"/>
-<pinref part="C5" gate="G$1" pin="1"/>
-<junction x="116.84" y="73.66"/>
-<pinref part="U4" gate="G$1" pin="VCC"/>
-<pinref part="SUPPLY1" gate="G$1" pin="5V"/>
-</segment>
-</net>
-<net name="N$2" class="0">
-<segment>
-<pinref part="IC1" gate="G$1" pin="PCINT12/OC0B/SS_PB4"/>
-<wire x1="0" y1="63.5" x2="-2.54" y2="63.5" width="0.1524" layer="91"/>
-</segment>
-</net>
-<net name="SCK" class="0">
-<segment>
-<wire x1="-17.78" y1="58.42" x2="-15.24" y2="55.88" width="0.1524" layer="91"/>
-<wire x1="-15.24" y1="55.88" x2="-2.54" y2="55.88" width="0.1524" layer="91"/>
-<label x="-15.24" y="55.88" size="1.778" layer="95"/>
 </segment>
 <segment>
@@
 <segment>
 <wire x1="-17.78" y1="66.04" x2="-15.24" y2="63.5" width="0.1524" layer="91"/>
-<wire x1="-15.24" y1="63.5" x2="-2.54" y2="63.5" width="0.1524" layer="91"/>
+<wire x1="-15.24" y1="63.5" x2="0" y2="63.5" width="0.1524" layer="91"/>
 <label x="-15.24" y="63.5" size="1.778" layer="95"/>
+<pinref part="IC1" gate="G$1" pin="PCINT12/OC0B/SS_PB4"/>
 </segment>
 </net>
@@
 <wire x1="185.42" y1="63.5" x2="182.88" y2="60.96" width="0.1524" layer="91"/>
 <label x="165.1" y="60.96" size="1.778" layer="95"/>
-</segment>
-</net>
-<net name="MOSI" class="0">
-<segment>
-<pinref part="IC1" gate="G$1" pin="PCINT13/MOSI_PB5"/>
-<wire x1="0" y1="60.96" x2="-15.24" y2="60.96" width="0.1524" layer="91"/>
-<wire x1="-15.24" y1="60.96" x2="-17.78" y2="63.5" width="0.1524" layer="91"/>
-<label x="-15.24" y="60.96" size="1.778" layer="95"/>
-</segment>
-</net>
-<net name="ID" class="0">
-<segment>
-<pinref part="J1" gate="G$1" pin="ID"/>
-<wire x1="-10.16" y1="-38.1" x2="-40.64" y2="-38.1" width="0.1524" layer="91"/>
-<wire x1="-40.64" y1="-38.1" x2="-43.18" y2="-35.56" width="0.1524" layer="91"/>
-<label x="-40.64" y="-38.1" size="1.778" layer="95"/>
 </segment>
 </net>
@@
 <wire x1="-45.72" y1="-30.48" x2="-43.18" y2="-27.94" width="0.1524" layer="91"/>
 <label x="-60.96" y="-30.48" size="1.778" layer="95"/>
+<junction x="-53.34" y="-30.48"/>
 </segment>
 </net>
@@
 </segment>
 </net>
-<net name="N$11" class="0">
-<segment>
-<wire x1="218.44" y1="157.48" x2="218.44" y2="-99.06" width="0.1524" layer="91" style="shortdash"/>
-</segment>
-</net>
 <net name="N$13" class="0">
 <segment>
@@
 <pinref part="J2" gate="G$1" pin="1"/>
 <label x="309.88" y="50.8" size="1.778" layer="95"/>
+<junction x="307.34" y="48.26"/>
 </segment>
 </net>
@@
 <wire x1="198.12" y1="25.4" x2="198.12" y2="22.86" width="0.1524" layer="91"/>
 <wire x1="203.2" y1="25.4" x2="198.12" y2="25.4" width="0.1524" layer="91"/>
+<junction x="198.12" y="25.4"/>
 </segment>
 </net>
@@
 </sheet>
 </sheets>
+<errors>
+</errors>
 </schematic>
 </drawing>
