File: Reflow-A-Tron/Reflow-A-Tron.sch (EAGLE design)
At the start: 41 parts, among them IC1 ATMEGA644-10PU, J2 HOT, J3 NEUTRAL, Q1 FOXSLF/200-20, Q2 BSS123, U1 FT230X, U2 L4941BDT-TRDPAK-3, U4 MAX6675

Commit message: Next rev with more bug fixes
Other:
- moved on the sheet: C5, C6
Changed lines of the file:
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@@
 <instance part="C2" gate="G$1" x="33.02" y="121.92"/>
 <instance part="GND3" gate="1" x="106.68" y="60.96"/>
-<instance part="C5" gate="G$1" x="116.84" y="68.58"/>
+<instance part="C5" gate="G$1" x="116.84" y="71.12" rot="R180"/>
 <instance part="S1" gate="S" x="-53.34" y="60.96"/>
 <instance part="GND4" gate="1" x="-58.42" y="53.34"/>
-<instance part="C6" gate="G$1" x="-55.88" y="33.02"/>
+<instance part="C6" gate="G$1" x="-55.88" y="35.56" rot="R180"/>
 <instance part="SUPPLY6" gate="G$1" x="-60.96" y="40.64"/>
 <instance part="Q1" gate="G$1" x="-58.42" y="10.16"/>
@@
 <wire x1="-60.96" y1="40.64" x2="-60.96" y2="38.1" width="0.1524" layer="91"/>
 <pinref part="C6" gate="G$1" pin="1"/>
-<wire x1="-55.88" y1="30.48" x2="-48.26" y2="38.1" width="0.1524" layer="91"/>
+<wire x1="-55.88" y1="38.1" x2="-48.26" y2="38.1" width="0.1524" layer="91"/>
 <label x="-48.26" y="38.1" size="1.778" layer="95"/>
-<wire x1="-60.96" y1="38.1" x2="-55.88" y2="30.48" width="0.1524" layer="91"/>
-<junction x="-55.88" y="30.48"/>
+<wire x1="-60.96" y1="38.1" x2="-55.88" y2="38.1" width="0.1524" layer="91"/>
+<junction x="-55.88" y="38.1"/>
 </segment>
 <segment>
@@
 </segment>
 <segment>
-<wire x1="116.84" y1="78.74" x2="116.84" y2="66.04" width="0.1524" layer="91"/>
-<wire x1="116.84" y1="66.04" x2="124.46" y2="73.66" width="0.1524" layer="91"/>
+<wire x1="116.84" y1="78.74" x2="116.84" y2="73.66" width="0.1524" layer="91"/>
+<wire x1="116.84" y1="73.66" x2="124.46" y2="73.66" width="0.1524" layer="91"/>
 <pinref part="C5" gate="G$1" pin="1"/>
-<junction x="116.84" y="66.04"/>
+<junction x="116.84" y="73.66"/>
 <pinref part="U4" gate="G$1" pin="VCC"/>
 <pinref part="SUPPLY1" gate="G$1" pin="5V"/>
@@
 <segment>
 <pinref part="GND3" gate="1" pin="GND"/>
-<wire x1="124.46" y1="66.04" x2="116.84" y2="71.12" width="0.1524" layer="91"/>
-<wire x1="116.84" y1="71.12" x2="106.68" y2="66.04" width="0.1524" layer="91"/>
 <wire x1="106.68" y1="66.04" x2="106.68" y2="63.5" width="0.1524" layer="91"/>
+<pinref part="U4" gate="G$1" pin="GND"/>
+<wire x1="124.46" y1="66.04" x2="116.84" y2="66.04" width="0.1524" layer="91"/>
 <pinref part="C5" gate="G$1" pin="2"/>
-<junction x="116.84" y="71.12"/>
-<pinref part="U4" gate="G$1" pin="GND"/>
+<wire x1="116.84" y1="66.04" x2="106.68" y2="66.04" width="0.1524" layer="91"/>
+<wire x1="116.84" y1="66.04" x2="116.84" y2="68.58" width="0.1524" layer="91"/>
+<junction x="116.84" y="66.04"/>
 </segment>
 <segment>
@@
 <segment>
 <pinref part="C6" gate="G$1" pin="2"/>
-<wire x1="-55.88" y1="35.56" x2="-48.26" y2="30.48" width="0.1524" layer="91"/>
-<wire x1="-55.88" y1="35.56" x2="-60.96" y2="30.48" width="0.1524" layer="91"/>
-<label x="-48.26" y="30.48" size="1.778" layer="95"/>
+<wire x1="-55.88" y1="33.02" x2="-48.26" y2="33.02" width="0.1524" layer="91"/>
+<wire x1="-55.88" y1="33.02" x2="-60.96" y2="33.02" width="0.1524" layer="91"/>
+<label x="-48.26" y="33.02" size="1.778" layer="95"/>
 <pinref part="GND10" gate="1" pin="GND"/>
-<wire x1="-60.96" y1="30.48" x2="-60.96" y2="27.94" width="0.1524" layer="91"/>
-<junction x="-55.88" y="35.56"/>
-</segment>
-<segment>
+<wire x1="-60.96" y1="33.02" x2="-60.96" y2="27.94" width="0.1524" layer="91"/>
+<junction x="-55.88" y="33.02"/>
+</segment>
+<segment>

Commit message: Hardware Working for reflow a tron
Parts:
- removed C9: 10nF, neilbetham:SMD-CAP-0805
- removed D3: (no value), neilbetham:T1250H
- added D5: HV TRIAC, custom:T1250H
- C5: value 10nF -> 100nF
- J1: value (none) -> USB Mini
- J2: value HOT -> LINE
- J3: value NEUTRAL -> LOAD
Connections:
- removed net T-: C9.1, THERMOCOUPLE.2, U4.T-
- net GND: now also THERMOCOUPLE.2, U4.T-
- net HOT: now also D5.A2; no longer D3.A2
- net N$14: now also D5.G; no longer D3.G
- net NEUTRAL: now also D5.A1; no longer D3.A1
- net T+: no longer C9.2
Other:
- moved on the sheet: J1
Changed lines of the file:
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@@
 <part name="C2" library="SparkFun-Capacitors" deviceset="10UF50V20%(1210)" device="" value="10uF"/>
 <part name="GND3" library="SparkFun-Aesthetics" deviceset="GND" device=""/>
-<part name="C5" library="custom" deviceset="SMD-CAP" device="-0805" value="10nF"/>
+<part name="C5" library="custom" deviceset="SMD-CAP" device="-0805" value="100nF"/>
 <part name="S1" library="SparkFun-Retired" deviceset="TAC_SWITCH" device="PTH"/>
 <part name="GND4" library="SparkFun-Aesthetics" deviceset="GND" device=""/>
@@
 <part name="C7" library="neilbetham" deviceset="SMD-CAP" device="-0805" value="36pF"/>
 <part name="C8" library="neilbetham" deviceset="SMD-CAP" device="-0805" value="36pF"/>
-<part name="C9" library="neilbetham" deviceset="SMD-CAP" device="-0805" value="10nF"/>
 <part name="R2" library="resistor" deviceset="R-US_" device="R0805" value="10k"/>
 <part name="R1" library="resistor" deviceset="R-US_" device="R0805" value="10k"/>
@@
 <part name="GND7" library="SparkFun-Aesthetics" deviceset="GND" device=""/>
 <part name="U1" library="custom" deviceset="FT230X" device="" value="FT230X"/>
-<part name="J1" library="custom" deviceset="XM7D-0512" device=""/>
 <part name="GND8" library="SparkFun-Aesthetics" deviceset="GND" device=""/>
 <part name="C3" library="neilbetham" deviceset="SMD-CAP" device="-0805" value="100nF"/>
@@
 <part name="GND6" library="SparkFun-Aesthetics" deviceset="GND" device=""/>
 <part name="SUPPLY5" library="SparkFun-Aesthetics" deviceset="5V" device=""/>
-<part name="D3" library="neilbetham" deviceset="T1250H" device=""/>
 <part name="OK1" library="optocoupler" deviceset="IL420" device=""/>
 <part name="R8" library="resistor" deviceset="R-US_" device="R0805" value="180"/>
@@
 <part name="R11" library="resistor" deviceset="R-US_" device="R0805" value="150"/>
 <part name="Q2" library="transistor-small-signal" deviceset="BSS123" device=""/>
-<part name="J2" library="neilbetham" deviceset="8191" device="" value="HOT"/>
-<part name="J3" library="neilbetham" deviceset="8191" device="" value="NEUTRAL"/>
+<part name="J2" library="neilbetham" deviceset="8191" device="" value="LINE"/>
+<part name="J3" library="neilbetham" deviceset="8191" device="" value="LOAD"/>
 <part name="GND10" library="SparkFun-Aesthetics" deviceset="GND" device=""/>
 <part name="R12" library="resistor" deviceset="R-US_" device="R0805" value="10k"/>
 <part name="GND5" library="SparkFun-Aesthetics" deviceset="GND" device=""/>
+<part name="GND9" library="SparkFun-Aesthetics" deviceset="GND" device=""/>
+<part name="J1" library="custom" deviceset="XM7D-0512" device="" value="USB Mini"/>
+<part name="D5" library="custom" deviceset="T1250H" device="" value="HV TRIAC"/>
 </parts>
 <sheets>
@@
 <instance part="C7" gate="G$1" x="-63.5" y="5.08"/>
 <instance part="C8" gate="G$1" x="-53.34" y="5.08"/>
-<instance part="C9" gate="G$1" x="121.92" y="43.18"/>
 <instance part="R2" gate="G$1" x="165.1" y="81.28" rot="R270"/>
 <instance part="R1" gate="G$1" x="149.86" y="43.18" rot="R270"/>
@@
 <instance part="GND7" gate="1" x="63.5" y="119.38"/>
 <instance part="U1" gate="G$1" x="43.18" y="-35.56"/>
-<instance part="J1" gate="G$1" x="-10.16" y="-35.56"/>
 <instance part="GND8" gate="1" x="25.4" y="-53.34"/>
 <instance part="C3" gate="G$1" x="25.4" y="-40.64"/>
@@
 <instance part="GND6" gate="1" x="175.26" y="-17.78"/>
 <instance part="SUPPLY5" gate="G$1" x="165.1" y="5.08"/>
-<instance part="D3" gate="G$1" x="307.34" y="35.56" rot="MR0"/>
 <instance part="OK1" gate="G$1" x="220.98" y="35.56"/>
 <instance part="R8" gate="G$1" x="251.46" y="48.26"/>
@@
 <instance part="R12" gate="G$1" x="190.5" y="7.62" rot="R270"/>
 <instance part="GND5" gate="1" x="195.58" y="-5.08"/>
+<instance part="GND9" gate="1" x="121.92" y="30.48"/>
+<instance part="J1" gate="G$1" x="-7.62" y="-35.56"/>
+<instance part="D5" gate="G$1" x="307.34" y="35.56" rot="MR0"/>
 </instances>
 <busses>
@@
 </segment>
 <segment>
-<pinref part="J1" gate="G$1" pin="GND"/>
-<wire x1="-10.16" y1="-40.64" x2="-40.64" y2="-40.64" width="0.1524" layer="91"/>
+<wire x1="-7.62" y1="-40.64" x2="-40.64" y2="-40.64" width="0.1524" layer="91"/>
 <wire x1="-40.64" y1="-40.64" x2="-43.18" y2="-38.1" width="0.1524" layer="91"/>
 <label x="-40.64" y="-40.64" size="1.778" layer="95"/>
@@
 <label x="-60.96" y="-43.18" size="1.778" layer="95"/>
 <junction x="-53.34" y="-40.64"/>
+<pinref part="J1" gate="G$1" pin="GND"/>
 </segment>
 <segment>
@@
 <label x="63.5" y="50.8" size="1.778" layer="95"/>
 </segment>
+<segment>
+<wire x1="124.46" y1="60.96" x2="114.3" y2="60.96" width="0.1524" layer="91"/>
+<wire x1="114.3" y1="60.96" x2="114.3" y2="40.64" width="0.1524" layer="91"/>
+<pinref part="U4" gate="G$1" pin="T-"/>
+<wire x1="114.3" y1="40.64" x2="121.92" y2="40.64" width="0.1524" layer="91"/>
+<wire x1="121.92" y1="40.64" x2="129.54" y2="40.64" width="0.1524" layer="91"/>
+<wire x1="129.54" y1="40.64" x2="129.54" y2="43.18" width="0.1524" layer="91"/>
+<pinref part="THERMOCOUPLE" gate="G$1" pin="2"/>
+<wire x1="129.54" y1="43.18" x2="132.08" y2="43.18" width="0.1524" layer="91"/>
+<pinref part="GND9" gate="1" pin="GND"/>
+<wire x1="121.92" y1="40.64" x2="121.92" y2="33.02" width="0.1524" layer="91"/>
+<junction x="121.92" y="40.64"/>
+</segment>
 </net>
 <net name="RESET" class="0">
@@
 <wire x1="124.46" y1="58.42" x2="116.84" y2="58.42" width="0.1524" layer="91"/>
 <wire x1="116.84" y1="58.42" x2="116.84" y2="45.72" width="0.1524" layer="91"/>
-<pinref part="C9" gate="G$1" pin="2"/>
-<wire x1="116.84" y1="45.72" x2="121.92" y2="45.72" width="0.1524" layer="91"/>
 <pinref part="U4" gate="G$1" pin="T+"/>
 <pinref part="THERMOCOUPLE" gate="G$1" pin="1"/>
-<wire x1="121.92" y1="45.72" x2="132.08" y2="45.72" width="0.1524" layer="91"/>
-<junction x="121.92" y="45.72"/>
-</segment>
-</net>
-<net name="T-" class="0">
-<segment>
-<wire x1="124.46" y1="60.96" x2="114.3" y2="60.96" width="0.1524" layer="91"/>
-<wire x1="114.3" y1="60.96" x2="114.3" y2="40.64" width="0.1524" layer="91"/>
-<pinref part="C9" gate="G$1" pin="1"/>
-<wire x1="114.3" y1="40.64" x2="121.92" y2="40.64" width="0.1524" layer="91"/>
-<pinref part="U4" gate="G$1" pin="T-"/>
-<wire x1="121.92" y1="40.64" x2="129.54" y2="40.64" width="0.1524" layer="91"/>
-<wire x1="129.54" y1="40.64" x2="129.54" y2="43.18" width="0.1524" layer="91"/>
-<pinref part="THERMOCOUPLE" gate="G$1" pin="2"/>
-<wire x1="129.54" y1="43.18" x2="132.08" y2="43.18" width="0.1524" layer="91"/>
-<junction x="121.92" y="40.64"/>
+<wire x1="116.84" y1="45.72" x2="132.08" y2="45.72" width="0.1524" layer="91"/>
 </segment>
 </net>
@@
 <net name="USB-VCC" class="0">
 <segment>
-<pinref part="J1" gate="G$1" pin="VCC"/>
-<wire x1="-10.16" y1="-30.48" x2="-40.64" y2="-30.48" width="0.1524" layer="91"/>
+<wire x1="-7.62" y1="-30.48" x2="-40.64" y2="-30.48" width="0.1524" layer="91"/>
 <wire x1="-40.64" y1="-30.48" x2="-43.18" y2="-27.94" width="0.1524" layer="91"/>
 <label x="-40.64" y="-30.48" size="1.778" layer="95"/>
@@
 <label x="-60.96" y="-30.48" size="1.778" layer="95"/>
 <junction x="-53.34" y="-30.48"/>
+<pinref part="J1" gate="G$1" pin="VCC"/>
 </segment>
 </net>
@@
 <segment>
 <pinref part="R4" gate="G$1" pin="2"/>
+<wire x1="-25.4" y1="-35.56" x2="-7.62" y2="-35.56" width="0.1524" layer="91"/>
 <pinref part="J1" gate="G$1" pin="DM"/>
-<wire x1="-25.4" y1="-35.56" x2="-10.16" y2="-35.56" width="0.1524" layer="91"/>
 </segment>
 </net>
@@
 <segment>
 <pinref part="R3" gate="G$1" pin="2"/>
+<wire x1="-12.7" y1="-33.02" x2="-7.62" y2="-33.02" width="0.1524" layer="91"/>
 <pinref part="J1" gate="G$1" pin="DP"/>
-<wire x1="-12.7" y1="-33.02" x2="-10.16" y2="-33.02" width="0.1524" layer="91"/>
 </segment>
 </net>
@@
 <pinref part="OK1" gate="G$1" pin="A1"/>
 <wire x1="231.14" y1="33.02" x2="287.02" y2="33.02" width="0.1524" layer="91"/>
-<pinref part="D3" gate="G$1" pin="G"/>
 <pinref part="R10" gate="G$1" pin="2"/>
 <wire x1="287.02" y1="33.02" x2="298.831" y2="33.02" width="0.1524" layer="91"/>
 <wire x1="287.02" y1="27.94" x2="287.02" y2="33.02" width="0.1524" layer="91"/>
 <junction x="287.02" y="33.02"/>
+<pinref part="D5" gate="G$1" pin="G"/>
 </segment>
 </net>
@@
 <pinref part="R9" gate="G$1" pin="2"/>
 <wire x1="284.48" y1="48.26" x2="307.34" y2="48.26" width="0.1524" layer="91"/>
-<pinref part="D3" gate="G$1" pin="A2"/>
 <wire x1="307.34" y1="48.26" x2="314.96" y2="48.26" width="0.1524" layer="91"/>
 <wire x1="307.34" y1="43.18" x2="307.34" y2="48.26" width="0.1524" layer="91"/>
@@
 <label x="309.88" y="50.8" size="1.778" layer="95"/>
 <junction x="307.34" y="48.26"/>
+<pinref part="D5" gate="G$1" pin="A2"/>
 </segment>
 </net>
@@
 <wire x1="307.34" y1="15.24" x2="314.96" y2="15.24" width="0.1524" layer="91"/>
 <wire x1="287.02" y1="17.78" x2="287.02" y2="15.24" width="0.1524" layer="91"/>
-<pinref part="D3" gate="G$1" pin="A1"/>
 <wire x1="307.34" y1="29.21" x2="307.34" y2="15.24" width="0.1524" layer="91"/>
 <junction x="287.02" y="15.24"/>
@@
 <pinref part="J3" gate="G$1" pin="1"/>
 <label x="302.26" y="10.16" size="1.778" layer="95"/>
-</segment>
-</net>
+<pinref part="D5" gate="G$1" pin="A1"/>
+</segment>
+</net>
